File: hardware/led aquário.kicad_pcb (KiCad board)
At the start: 2 copper layers, 98.7 x 100.5 mm, 50 parts, among them J1 Conn_01x01, J2 Conn_01x01, J3 Conn_01x01, J4 Conn_01x01, J5 Conn_01x01, J6 Conn_01x01, J7 Conn_01x01, J8 Conn_01x01

Commit message: att
Parts:
- J1, J2, J3, J4, J5, J6, J7, J8: footprint TestPoint:TestPoint_THTPad_4.0x4.0mm_Drill2.0mm -> TestPoint:TestPoint_Pad_4.0x4.0mm
- R1, R10, R11, R12, R13, R14, R2, R3, R4, R5, R6, R7, R8, R9: footprint Resistor_SMD:R_1206_3216Metric -> Resistor_SMD:R_2512_6332Metric
- moved R1 70.9 mm to (301.5, 168.0)
- moved R2 70.5 mm to (301.5, 172.9)
- moved R12 69.2 mm to (301.5, 103.4)
- moved R11 68.8 mm to (301.5, 98.5)
- moved R3 43.0 mm to (301.5, 154.0)
- moved R4 42.6 mm to (301.5, 158.9)
- moved R10 41.5 mm to (301.0, 116.9)
- moved R9 41.0 mm to (301.0, 112.0)
- moved J1 22.8 mm to (294.0, 121.0)
- moved R5 19.8 mm to (301.5, 145.0)
- moved J6 14.4 mm to (294.5, 163.0)
- moved R8 14.3 mm to (301.0, 130.4)
- moved R7 13.9 mm to (301.0, 125.5)
- moved R6 9.53 mm to (301.5, 140.0)
- moved J4 6.01 mm to (294.5, 177.5)
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Connections:
- R1 pad 2: Net-(D4-K) -> Net-(D21-K)
- R10 pad 2: Net-(D17-K) -> Net-(D5-K)
- R11 pad 2: Net-(D21-K) -> Net-(D4-K)
- R12 pad 2: Net-(D21-K) -> Net-(D4-K)
- R2 pad 2: Net-(D4-K) -> Net-(D21-K)
- R3 pad 2: Net-(D5-K) -> Net-(D17-K)
- R4 pad 2: Net-(D5-K) -> Net-(D17-K)
- R5 pad 2: Net-(D9-K) -> Net-(D13-K)
- R6 pad 2: Net-(D9-K) -> Net-(D13-K)
- R7 pad 2: Net-(D13-K) -> Net-(D9-K)
- R8 pad 2: Net-(D13-K) -> Net-(D9-K)
- R9 pad 2: Net-(D17-K) -> Net-(D5-K)
Routing:
- net Net-(D5-K): track 10.9 -> 16.4 mm
- net Net-(D9-K): track 11.5 -> 16.3 mm
- net Net-(D4-K): track 11.2 -> 15.4 mm
- net Net-(D13-K): track 11.7 -> 15.5 mm
- net Net-(D17-K): track 12.0 -> 15.3 mm
- net Net-(D25-K): track 11.3 -> 14.6 mm
- net Net-(D21-K): track 12.4 -> 15.4 mm
